File: 1.kicad_sch (KiCad schematic)
At the start: 40 parts, among them J1 Bat, J10 Conn_01x04_Pin, J11 TH, J2 Conn_01x04_Pin, J3 LED_pins, J4 USB_C, J5 Conn_GPIO, J6 Conn_GND, J7 Conn_3V3, J8 Conn_JTAG, J9 Conn_01x04_Pin, SW1 SW_Push, SW2 SW_Push, SW3 SW_DPDT_x2, U2 MCP73871, U3 XC6210B332MR

Commit message: Add files via upload
Parts:
- renumbered ESP32-C6-WROOM-1U to ESP32-C6-WROOM-1U1
Changed lines of the file:
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@@
 		(dnp no)
 		(fields_autoplaced yes)
-		(property "Reference" "ESP32-C6-WROOM-1U"
+		(property "Reference" "ESP32-C6-WROOM-1U1"
 			(at 193.9133 22.86 0)
 			(show_name no)
@@
 			(project "1"
 				(path "/8a57ca9b-e87d-4c78-8cca-6754fc21c15c"
-					(reference "ESP32-C6-WROOM-1U")
+					(reference "ESP32-C6-WROOM-1U1")
 					(unit 1)
 				)
